Commit message: Updated toycar.urdf
Added Lidar Sensor

File: urdf/toycar.urdf (robot description, URDF)
Before this commit: robot toycar, 7 links, 6 joints
Links:
- added link base_laser, mass 0.15717; collision mesh filename=package://toycar/meshes/ydlidar.dae; visual mesh filename=package://toycar/meshes/ydlidar.dae
Joints:
- added joint laser_joint: type continuous, parent chassis, child base_laser, origin xyz=0 0 0.2 rpy=0 0 0, axis 0 0 1
